File: supercrisp/keyboard_matrix.kicad_sch (KiCad schematic)
At the start: 89 parts, among them SW1 SW_Push, SW10 SW_Push, SW11 SW_Push, SW12 SW_Push, SW13 SW_Push, SW14 SW_Push, SW15 SW_Push, SW16 SW_Push, SW17 SW_Push, SW18 SW_Push, SW19 SW_Push, SW2 SW_Push, SW20 SW_Push, SW21 SW_Push, SW22 SW_Push, SW23 SW_Push, SW24 SW_Push, SW25 SW_Push, SW26 SW_Push, SW3 SW_Push, SW4 SW_Push, SW5 SW_Push, SW6 SW_Push, SW7 SW_Push, SW8 SW_Push, SW9 SW_Push

Commit message: WIP 0 errors, 58 warnings
Parts:
- renumbered COL0 to COL1, COL1 to COL2, COL2 to COL3, COL3 to COL4, COL4 to COL5, COL5 to COL6, D50 to D10, D3 to D11, D15 to D12, D27 to D13, D39 to D14, D51 to D15, D4 to D16, D16 to D17, D28 to D18, D40 to D19, D13 to D2, D52 to D20, D5 to D21, D17 to D22, D29 to D23, D41 to D24, D6 to D25, D18 to D26, D30 to D27, D42 to D28, D7 to D29, D25 to D3, D19 to D30, D43 to D32, D8 to D33, D20 to D34, D32 to D35, D44 to D36, D9 to D37, D21 to D38, D33 to D39, D37 to D4, D45 to D40, D10 to D41, D22 to D42, D34 to D43, D46 to D44, D11 to D45, D23 to D46, D35 to D47, D47 to D48, D12 to D49, D49 to D5, D24 to D50, D36 to D51, D48 to D52, D2 to D6, D14 to D7, D26 to D8, D38 to D9, ROW0 to ROW1, ROW1 to ROW2, ROW2 to ROW3, ROW3 to ROW4, ROW4 to ROW5, SW20 to SW10, SW26 to SW11, SW3 to SW12, SW9 to SW13, SW15 to SW14, SW21 to SW15, SW4 to SW16, SW10 to SW17, SW16 to SW18, SW22 to SW19, SW1 to SW2, SW5 to SW20, SW11 to SW21, SW17 to SW22, SW6 to SW24, SW12 to SW25, SW18 to SW26, SW24 to SW27, SW7 to SW3, SW13 to SW4, SW19 to SW5, SW25 to SW6, SW2 to SW7, SW14 to SW9

Commit message: Add JLPCB part numbers
Parts:
- COL1, COL2, COL3, COL4, COL5, COL6, ROW1, ROW2, ROW3, ROW4, ROW5, SW10, SW11, SW12, SW13, SW14, SW15, SW16, SW17, SW18, SW19, SW2, SW20, SW21, SW22, SW23, SW24, SW25, SW26, SW27, SW3, SW4, SW5, SW6, SW7, SW8, SW9: JLCPCB Part # (none) -> N/A
Changed lines of the file:
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@@
 			)
 		)
-		(property "JLCPCB Part #" ""
+		(property "JLCPCB Part #" "N/A"
 			(at 95.25 62.23 0)
 			(effects
@@
 			)
 		)
-		(property "JLCPCB Part #" ""
+		(property "JLCPCB Part #" "N/A"
 			(at 191.77 30.48 0)
 			(effects
@@
 			)
 		)
-		(property "JLCPCB Part #" ""
+		(property "JLCPCB Part #" "N/A"
 			(at 76.2 53.34 0)
 			(effects
@@
 			)
 		)
-		(property "JLCPCB Part #" ""
+		(property "JLCPCB Part #" "N/A"
 			(at 95.25 86.36 0)
 			(effects
@@
 			)
 		)
-		(property "JLCPCB Part #" ""
+		(property "JLCPCB Part #" "N/A"
 			(at 137.16 38.1 0)
 			(effects
@@
 			)
 		)
-		(property "JLCPCB Part #" ""
+		(property "JLCPCB Part #" "N/A"
 			(at 115.57 38.1 0)
 			(effects
@@
 			)
 		)
-		(property "JLCPCB Part #" ""
+		(property "JLCPCB Part #" "N/A"
 			(at 176.53 86.36 0)
 			(effects
@@
 			)
 		)
-		(property "JLCPCB Part #" ""
+		(property "JLCPCB Part #" "N/A"
 			(at 157.48 62.23 0)
 			(effects
@@
 			)
 		)
-		(property "JLCPCB Part #" ""
+		(property "JLCPCB Part #" "N/A"
 			(at 157.48 86.36 0)
 			(effects
@@
 			)
 		)
-		(property "JLCPCB Part #" ""
+		(property "JLCPCB Part #" "N/A"
 			(at 115.57 110.49 0)
 			(effects
@@
 			)
 		)
-		(property "JLCPCB Part #" ""
+		(property "JLCPCB Part #" "N/A"
 			(at 76.2 77.47 0)
 			(effects
@@
 			)
 		)
-		(property "JLCPCB Part #" ""
+		(property "JLCPCB Part #" "N/A"
 			(at 95.25 38.1 0)
 			(effects
@@
 			)
 		)
-		(property "JLCPCB Part #" ""
+		(property "JLCPCB Part #" "N/A"
 			(at 90.17 30.48 0)
 			(effects
@@
 			)
 		)
-		(property "JLCPCB Part #" ""
+		(property "JLCPCB Part #" "N/A"
 			(at 196.85 110.49 0)
 			(effects
@@
 			)
 		)
-		(property "JLCPCB Part #" ""
+		(property "JLCPCB Part #" "N/A"
 			(at 95.25 134.62 0)
 			(effects
@@
 			)
 		)
-		(property "JLCPCB Part #" ""
+		(property "JLCPCB Part #" "N/A"
 			(at 196.85 62.23 0)
 			(effects
@@
 			)
 		)
-		(property "JLCPCB Part #" ""
+		(property "JLCPCB Part #" "N/A"
 			(at 115.57 86.36 0)
 			(effects
@@
 			)
 		)
-		(property "JLCPCB Part #" ""
+		(property "JLCPCB Part #" "N/A"
 			(at 137.16 86.36 0)
 			(effects
@@
 			)
 		)
-		(property "JLCPCB Part #" ""
+		(property "JLCPCB Part #" "N/A"
 			(at 157.48 110.49 0)
 			(effects
@@
 			)
 		)
-		(property "JLCPCB Part #" ""
+		(property "JLCPCB Part #" "N/A"
 			(at 137.16 62.23 0)
 			(effects
@@
 			)
 		)
-		(property "JLCPCB Part #" ""
+		(property "JLCPCB Part #" "N/A"
 			(at 176.53 62.23 0)
 			(effects
@@
 			)
 		)
-		(property "JLCPCB Part #" ""
+		(property "JLCPCB Part #" "N/A"
 			(at 115.57 134.62 0)
 			(effects
@@
 			)
 		)
-		(property "JLCPCB Part #" ""
+		(property "JLCPCB Part #" "N/A"
 			(at 176.53 110.49 0)
 			(effects
@@
 			)
 		)
-		(property "JLCPCB Part #" ""
+		(property "JLCPCB Part #" "N/A"
 			(at 95.25 110.49 0)
 			(effects
@@
 			)
 		)
-		(property "JLCPCB Part #" ""
+		(property "JLCPCB Part #" "N/A"
 			(at 176.53 38.1 0)
 			(effects
@@
 			)
 		)
-		(property "JLCPCB Part #" ""
+		(property "JLCPCB Part #" "N/A"
 			(at 152.4 30.48 0)
 			(effects
@@
 			)
 		)
-		(property "JLCPCB Part #" ""
+		(property "JLCPCB Part #" "N/A"
 			(at 196.85 38.1 0)
 			(effects
@@
 			)
 		)
-		(property "JLCPCB Part #" ""
+		(property "JLCPCB Part #" "N/A"
 			(at 76.2 149.86 0)
 			(effects
@@
 			)
 		)
-		(property "JLCPCB Part #" ""
+		(property "JLCPCB Part #" "N/A"
 			(at 137.16 110.49 0)
 			(effects
@@
 			)
 		)
-		(property "JLCPCB Part #" ""
+		(property "JLCPCB Part #" "N/A"
 			(at 171.45 30.48 0)
 			(effects
@@
 			)
 		)
-		(property "JLCPCB Part #" ""
+		(property "JLCPCB Part #" "N/A"
 			(at 76.2 125.73 0)
 			(effects
@@
 			)
 		)
-		(property "JLCPCB Part #" ""
+		(property "JLCPCB Part #" "N/A"
 			(at 110.49 30.48 0)
 			(effects
@@
 			)
 		)
-		(property "JLCPCB Part #" ""
+		(property "JLCPCB Part #" "N/A"
 			(at 76.2 101.6 0)
 			(effects
@@
 			)
 		)
-		(property "JLCPCB Part #" ""
+		(property "JLCPCB Part #" "N/A"
 			(at 132.08 30.48 0)
 			(effects
@@
 			)
 		)
-		(property "JLCPCB Part #" ""
+		(property "JLCPCB Part #" "N/A"
 			(at 115.57 62.23 0)
 			(effects
@@
 			)
 		)
-		(property "JLCPCB Part #" ""
+		(property "JLCPCB Part #" "N/A"
 			(at 196.85 86.36 0)
 			(effects
@@
 			)
 		)
-		(property "JLCPCB Part #" ""
+		(property "JLCPCB Part #" "N/A"
 			(at 157.48 38.1 0)
 			(effects
