File: supercrisp/mcu.kicad_sch (KiCad schematic)
At the start: 14 parts, among them J1 SWD, J4 AudioJack4, SW1 SW_SPDT

Commit message: Add JLPCB part numbers
Parts:
- SW1: JLCPCB Part # (none) -> C221841
- USB_P1: JLCPCB Part # C319148 -> C319148
Changed lines of the file:
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@@
 			)
 		)
-		(property "JLCPCB Part #" "    C319148"
+		(property "JLCPCB Part #" "C319148"
 			(at 110.49 76.2 0)
 			(effects
@@
 			)
 		)
-		(property "JLCPCB Part #" ""
+		(property "JLCPCB Part #" "C221841"
 			(at 217.17 146.05 0)
 			(effects
