File: supercrisp/supercrisp.kicad_sch (KiCad schematic)
At the start: 6 parts

Commit message: Temp placement of switches and usb circuitry
Parts:
- added H7: MountingHole_Pad, MountingHole_NoSilkscreen:MountingHole_2.7mm_M2.5_DIN965_Pad_reversible, symbol Mechanical:MountingHole_Pad
Connections:
- net GND: now also H7.1

Commit message: WIP 0 errors, 58 warnings
Parts:
- added 3V3_TP1, BOOT0_TP1, NRST_TP1, SWCLK_TP1, SWDIO_TP1, USART_TP1, USB_CONN_DN_TP1, USB_CONN_DP_TP1, USB_DN_TP1, USB_DP_TP1, VBUS_TP1: TestPoint_Small, Testpoint_Rev:TestPoint_THTPad_D1.0mm_Drill0.5mm_reversible, symbol Connector:TestPoint_Small
- added C1, C3: 22uF, Capacitor_SMD:C_0603_1608Metric_Pad1.08x0.95mm_HandSolder, symbol Device:C_Small
- added C2: 430pF, Capacitor_SMD:C_0603_1608Metric_Pad1.08x0.95mm_HandSolder, symbol Device:C_Small
- added R1, R4: 100k, Resistor_SMD:R_0603_1608Metric, symbol Device:R_Small
- added R3: 309k, Resistor_SMD:R_0603_1608Metric, symbol Device:R_Small
- added U1: TPS82140, Package_LGA:Texas_SIL0008D_MicroSiP-8-1EP_2.8x3mm_P0.65mm_EP1.1x1.9mm, symbol Regulator_Switching:TPS82140
- added USB_U1: USBLC6-2SC6, Package_TO_SOT_SMD:SOT-23-6, symbol STM32F4_REV2-rescue:USBLC6-2SC6-Power_Protection
Connections:
- net GND: now also C1.2, C2.2, C3.2, R4.2, U1.3 (GND), U1.9 (GND), USB_U1.2 (GND)
- new net: R3.2, R4.1, U1.6 (FB)
- new net: R1.2, U1.7 (PG)
- new net: C2.1, U1.8 (SS/TR)
- new net BOOT0: BOOT0_TP1.1
- new net NRST: NRST_TP1.1
- new net SWCLK: SWCLK_TP1.1
- new net SWDIO: SWDIO_TP1.1
- new net USART: USART_TP1.1
- new net USB_CONN_DN: USB_CONN_DN_TP1.1, USB_U1.1 (I/O1)
- new net USB_CONN_DP: USB_CONN_DP_TP1.1, USB_U1.3 (I/O2)
- new net USB_DN: USB_DN_TP1.1, USB_U1.6 (I/O1)
- new net USB_DP: USB_DP_TP1.1, USB_U1.4 (I/O2)
- new net VBUS: C1.1, U1.1 (EN), U1.2 (VIN), USB_U1.5 (VBUS), VBUS_TP1.1
- new net VOUT_3V3: 3V3_TP1.1, C3.1, R1.1, R3.1, U1.4 (VOUT), U1.5 (VOUT)
Other:
- sheet MCU_BOTTOM ports: added BOOT0, NRST, SWCLK, SWDIO, USART3_TX, USB_CONN_DN, USB_CONN_DP, USB_DN, USB_DP, VBUS, VOUT_3V3; removed none
- sheet MCU_TOP ports: added BOOT0, NRST, SWCLK, SWDIO, USART3_TX, USB_CONN_DN, USB_CONN_DP, USB_DN, USB_DP, VBUS, VOUT_3V3; removed none

Commit message: Add JLPCB part numbers
Parts:
- 3V3_TP1, BOOT0_TP1, H1, H2, H3, H4, H5, H6, H7, NRST_TP1, SWCLK_TP1, SWDIO_TP1, USART_TP1, USB_CONN_DN_TP1, USB_CONN_DP_TP1, USB_DN_TP1, USB_DP_TP1, VBUS_TP1: JLCPCB Part # (none) -> N/A
- USB_U1: JLCPCB Part # (none) -> C323793
Changed lines of the file:
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@@
 			)
 		)
-		(property "JLCPCB Part #" ""
+		(property "JLCPCB Part #" "N/A"
 			(at 222.25 143.51 0)
 			(effects
@@
 			)
 		)
-		(property "JLCPCB Part #" ""
+		(property "JLCPCB Part #" "N/A"
 			(at 260.35 134.62 0)
 			(effects
@@
 			)
 		)
-		(property "JLCPCB Part #" ""
+		(property "JLCPCB Part #" "N/A"
 			(at 222.25 154.94 0)
 			(effects
@@
 			)
 		)
-		(property "JLCPCB Part #" ""
+		(property "JLCPCB Part #" "N/A"
 			(at 260.35 149.86 0)
 			(effects
@@
 			)
 		)
-		(property "JLCPCB Part #" ""
+		(property "JLCPCB Part #" "N/A"
 			(at 260.35 129.54 0)
 			(effects
@@
 			)
 		)
-		(property "JLCPCB Part #" ""
+		(property "JLCPCB Part #" "N/A"
 			(at 222.25 135.89 0)
 			(effects
@@
 			)
 		)
-		(property "JLCPCB Part #" ""
+		(property "JLCPCB Part #" "N/A"
 			(at 222.25 151.13 0)
 			(effects
@@
 			)
 		)
-		(property "JLCPCB Part #" ""
+		(property "JLCPCB Part #" "N/A"
 			(at 222.25 147.32 0)
 			(effects
@@
 			)
 		)
-		(property "JLCPCB Part #" ""
+		(property "JLCPCB Part #" "N/A"
 			(at 222.25 121.92 0)
 			(effects
@@
 			)
 		)
-		(property "JLCPCB Part #" ""
+		(property "JLCPCB Part #" "N/A"
 			(at 260.35 124.46 0)
 			(effects
@@
 			)
 		)
-		(property "JLCPCB Part #" ""
+		(property "JLCPCB Part #" "N/A"
 			(at 222.25 139.7 0)
 			(effects
@@
 			)
 		)
-		(property "JLCPCB Part #" ""
+		(property "JLCPCB Part #" "N/A"
 			(at 222.25 132.08 0)
 			(effects
@@
 			)
 		)
-		(property "JLCPCB Part #" ""
+		(property "JLCPCB Part #" "N/A"
 			(at 260.35 154.94 0)
 			(effects
@@
 			)
 		)
-		(property "JLCPCB Part #" ""
+		(property "JLCPCB Part #" "N/A"
 			(at 260.35 144.78 0)
 			(effects
@@
 			)
 		)
-		(property "JLCPCB Part #" ""
+		(property "JLCPCB Part #" "N/A"
 			(at 260.35 139.7 0)
 			(effects
@@
 			)
 		)
-		(property "JLCPCB Part #" ""
+		(property "JLCPCB Part #" "C323793"
 			(at 144.78 170.18 0)
 			(effects
@@
 			)
 		)
-		(property "JLCPCB Part #" ""
+		(property "JLCPCB Part #" "N/A"
 			(at 222.25 158.75 0)
 			(effects
@@
 			)
 		)
-		(property "JLCPCB Part #" ""
+		(property "JLCPCB Part #" "N/A"
 			(at 222.25 127 0)
 			(effects
@@
 			)
 		)
-		(property "JLCPCB Part #" ""
+		(property "JLCPCB Part #" "N/A"
 			(at 222.25 162.56 0)
 			(effects
