File: pcb/orbiter-wired/keyboard_matrix.kicad_sch (KiCad schematic)
At the start: 89 parts, among them SW10 SW_Push, SW11 SW_Push, SW12 SW_Push, SW13 SW_Push, SW14 SW_Push, SW15 SW_Push, SW16 SW_Push, SW17 SW_Push, SW18 SW_Push, SW19 SW_Push, SW2 SW_Push, SW20 SW_Push, SW21 SW_Push, SW22 SW_Push, SW23 SW_Push, SW24 SW_Push, SW25 SW_Push, SW26 SW_Push, SW27 SW_Push, SW3 SW_Push, SW4 SW_Push, SW5 SW_Push, SW6 SW_Push, SW7 SW_Push, SW8 SW_Push, SW9 SW_Push

Commit message: Orbiter wired v1.0 gerber & cleanup of old project files
Parts:
- COL1, COL2, COL3, COL4, COL5, COL6, ROW1, ROW2, ROW3, ROW4, ROW5, SW10, SW11, SW12, SW13, SW14, SW15, SW16, SW17, SW18, SW19, SW2, SW20, SW21, SW22, SW23, SW24, SW25, SW26, SW27, SW3, SW4, SW5, SW6, SW7, SW8, SW9: JLCPCB Part # N/A -> (none)

Commit message: Change diode footprints 0603 -> SOD-323
Parts:
- D1, D10, D11, D12, D13, D14, D15, D16, D17, D18, D19, D2, D20, D21, D22, D23, D24, D25, D26, D27, D28, D29, D3, D30, D31, D32, D33, D34, D35, D36, D37, D38, D39, D4, D40, D41, D42, D43, D44, D45, D46, D47, D48, D49, D5, D50, D51, D52, D6, D7, D8, D9: footprint Diode:D_0603_1608Metric_Pad1.05x0.95mm_HandSolder -> Diode_SMD:D_SOD-323_HandSoldering
Changed lines of the file:
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@@
 			)
 		)
-		(property "Footprint" "Diode:D_0603_1608Metric_Pad1.05x0.95mm_HandSolder"
+		(property "Footprint" "Diode_SMD:D_SOD-323_HandSoldering"
 			(at 162.56 73.66 0)
 			(effects
@@
 			)
 		)
-		(property "Footprint" "Diode:D_0603_1608Metric_Pad1.05x0.95mm_HandSolder"
+		(property "Footprint" "Diode_SMD:D_SOD-323_HandSoldering"
 			(at 181.61 49.53 0)
 			(effects
@@
 			)
 		)
-		(property "Footprint" "Diode:D_0603_1608Metric_Pad1.05x0.95mm_HandSolder"
+		(property "Footprint" "Diode_SMD:D_SOD-323_HandSoldering"
 			(at 185.42 97.79 0)
 			(effects
@@
 			)
 		)
-		(property "Footprint" "Diode:D_0603_1608Metric_Pad1.05x0.95mm_HandSolder"
+		(property "Footprint" "Diode_SMD:D_SOD-323_HandSoldering"
 			(at 120.65 146.05 0)
 			(effects
@@
 			)
 		)
-		(property "Footprint" "Diode:D_0603_1608Metric_Pad1.05x0.95mm_HandSolder"
+		(property "Footprint" "Diode_SMD:D_SOD-323_HandSoldering"
 			(at 100.33 49.53 0)
 			(effects
@@
 			)
 		)
-		(property "Footprint" "Diode:D_0603_1608Metric_Pad1.05x0.95mm_HandSolder"
+		(property "Footprint" "Diode_SMD:D_SOD-323_HandSoldering"
 			(at 100.33 97.79 0)
 			(effects
@@
 			)
 		)
-		(property "Footprint" "Diode:D_0603_1608Metric_Pad1.05x0.95mm_HandSolder"
+		(property "Footprint" "Diode_SMD:D_SOD-323_HandSoldering"
 			(at 142.24 73.66 0)
 			(effects
@@
 			)
 		)
-		(property "Footprint" "Diode:D_0603_1608Metric_Pad1.05x0.95mm_HandSolder"
+		(property "Footprint" "Diode_SMD:D_SOD-323_HandSoldering"
 			(at 166.37 73.66 0)
 			(effects
@@
 			)
 		)
-		(property "Footprint" "Diode:D_0603_1608Metric_Pad1.05x0.95mm_HandSolder"
+		(property "Footprint" "Diode_SMD:D_SOD-323_HandSoldering"
 			(at 201.93 73.66 0)
 			(effects
@@
 			)
 		)
-		(property "Footprint" "Diode:D_0603_1608Metric_Pad1.05x0.95mm_HandSolder"
+		(property "Footprint" "Diode_SMD:D_SOD-323_HandSoldering"
 			(at 104.14 121.92 0)
 			(effects
@@
 			)
 		)
-		(property "Footprint" "Diode:D_0603_1608Metric_Pad1.05x0.95mm_HandSolder"
+		(property "Footprint" "Diode_SMD:D_SOD-323_HandSoldering"
 			(at 166.37 49.53 0)
 			(effects
@@
 			)
 		)
-		(property "Footprint" "Diode:D_0603_1608Metric_Pad1.05x0.95mm_HandSolder"
+		(property "Footprint" "Diode_SMD:D_SOD-323_HandSoldering"
 			(at 120.65 97.79 0)
 			(effects
@@
 			)
 		)
-		(property "Footprint" "Diode:D_0603_1608Metric_Pad1.05x0.95mm_HandSolder"
+		(property "Footprint" "Diode_SMD:D_SOD-323_HandSoldering"
 			(at 205.74 121.92 0)
 			(effects
@@
 			)
 		)
-		(property "Footprint" "Diode:D_0603_1608Metric_Pad1.05x0.95mm_HandSolder"
+		(property "Footprint" "Diode_SMD:D_SOD-323_HandSoldering"
 			(at 142.24 97.79 0)
 			(effects
@@
 			)
 		)
-		(property "Footprint" "Diode:D_0603_1608Metric_Pad1.05x0.95mm_HandSolder"
+		(property "Footprint" "Diode_SMD:D_SOD-323_HandSoldering"
 			(at 201.93 49.53 0)
 			(effects
@@
 			)
 		)
-		(property "Footprint" "Diode:D_0603_1608Metric_Pad1.05x0.95mm_HandSolder"
+		(property "Footprint" "Diode_SMD:D_SOD-323_HandSoldering"
 			(at 162.56 49.53 0)
 			(effects
@@
 			)
 		)
-		(property "Footprint" "Diode:D_0603_1608Metric_Pad1.05x0.95mm_HandSolder"
+		(property "Footprint" "Diode_SMD:D_SOD-323_HandSoldering"
 			(at 146.05 73.66 0)
 			(effects
@@
 			)
 		)
-		(property "Footprint" "Diode:D_0603_1608Metric_Pad1.05x0.95mm_HandSolder"
+		(property "Footprint" "Diode_SMD:D_SOD-323_HandSoldering"
 			(at 185.42 49.53 0)
 			(effects
@@
 			)
 		)
-		(property "Footprint" "Diode:D_0603_1608Metric_Pad1.05x0.95mm_HandSolder"
+		(property "Footprint" "Diode_SMD:D_SOD-323_HandSoldering"
 			(at 162.56 97.79 0)
 			(effects
@@
 			)
 		)
-		(property "Footprint" "Diode:D_0603_1608Metric_Pad1.05x0.95mm_HandSolder"
+		(property "Footprint" "Diode_SMD:D_SOD-323_HandSoldering"
 			(at 146.05 49.53 0)
 			(effects
@@
 			)
 		)
-		(property "Footprint" "Diode:D_0603_1608Metric_Pad1.05x0.95mm_HandSolder"
+		(property "Footprint" "Diode_SMD:D_SOD-323_HandSoldering"
 			(at 181.61 121.92 0)
 			(effects
@@
 			)
 		)
-		(property "Footprint" "Diode:D_0603_1608Metric_Pad1.05x0.95mm_HandSolder"
+		(property "Footprint" "Diode_SMD:D_SOD-323_HandSoldering"
 			(at 205.74 97.79 0)
 			(effects
@@
 			)
 		)
-		(property "Footprint" "Diode:D_0603_1608Metric_Pad1.05x0.95mm_HandSolder"
+		(property "Footprint" "Diode_SMD:D_SOD-323_HandSoldering"
 			(at 201.93 121.92 0)
 			(effects
@@
 			)
 		)
-		(property "Footprint" "Diode:D_0603_1608Metric_Pad1.05x0.95mm_HandSolder"
+		(property "Footprint" "Diode_SMD:D_SOD-323_HandSoldering"
 			(at 185.42 73.66 0)
 			(effects
@@
 			)
 		)
-		(property "Footprint" "Diode:D_0603_1608Metric_Pad1.05x0.95mm_HandSolder"
+		(property "Footprint" "Diode_SMD:D_SOD-323_HandSoldering"
 			(at 100.33 121.92 0)
 			(effects
@@
 			)
 		)
-		(property "Footprint" "Diode:D_0603_1608Metric_Pad1.05x0.95mm_HandSolder"
+		(property "Footprint" "Diode_SMD:D_SOD-323_HandSoldering"
 			(at 162.56 121.92 0)
 			(effects
@@
 			)
 		)
-		(property "Footprint" "Diode:D_0603_1608Metric_Pad1.05x0.95mm_HandSolder"
+		(property "Footprint" "Diode_SMD:D_SOD-323_HandSoldering"
 			(at 124.46 73.66 0)
 			(effects
@@
 			)
 		)
-		(property "Footprint" "Diode:D_0603_1608Metric_Pad1.05x0.95mm_HandSolder"
+		(property "Footprint" "Diode_SMD:D_SOD-323_HandSoldering"
 			(at 181.61 73.66 0)
 			(effects
@@
 			)
 		)
-		(property "Footprint" "Diode:D_0603_1608Metric_Pad1.05x0.95mm_HandSolder"
+		(property "Footprint" "Diode_SMD:D_SOD-323_HandSoldering"
 			(at 124.46 146.05 0)
 			(effects
@@
 			)
 		)
-		(property "Footprint" "Diode:D_0603_1608Metric_Pad1.05x0.95mm_HandSolder"
+		(property "Footprint" "Diode_SMD:D_SOD-323_HandSoldering"
 			(at 124.46 97.79 0)
 			(effects
@@
 			)
 		)
-		(property "Footprint" "Diode:D_0603_1608Metric_Pad1.05x0.95mm_HandSolder"
+		(property "Footprint" "Diode_SMD:D_SOD-323_HandSoldering"
 			(at 104.14 146.05 0)
 			(effects
@@
 			)
 		)
-		(property "Footprint" "Diode:D_0603_1608Metric_Pad1.05x0.95mm_HandSolder"
+		(property "Footprint" "Diode_SMD:D_SOD-323_HandSoldering"
 			(at 205.74 49.53 0)
 			(effects
@@
 			)
 		)
-		(property "Footprint" "Diode:D_0603_1608Metric_Pad1.05x0.95mm_HandSolder"
+		(property "Footprint" "Diode_SMD:D_SOD-323_HandSoldering"
 			(at 201.93 97.79 0)
 			(effects
@@
 			)
 		)
-		(property "Footprint" "Diode:D_0603_1608Metric_Pad1.05x0.95mm_HandSolder"
+		(property "Footprint" "Diode_SMD:D_SOD-323_HandSoldering"
 			(at 142.24 49.53 0)
 			(effects
@@
 			)
 		)
-		(property "Footprint" "Diode:D_0603_1608Metric_Pad1.05x0.95mm_HandSolder"
+		(property "Footprint" "Diode_SMD:D_SOD-323_HandSoldering"
 			(at 146.05 121.92 0)
 			(effects
@@
 			)
 		)
-		(property "Footprint" "Diode:D_0603_1608Metric_Pad1.05x0.95mm_HandSolder"
+		(property "Footprint" "Diode_SMD:D_SOD-323_HandSoldering"
 			(at 120.65 73.66 0)
 			(effects
@@
 			)
 		)
-		(property "Footprint" "Diode:D_0603_1608Metric_Pad1.05x0.95mm_HandSolder"
+		(property "Footprint" "Diode_SMD:D_SOD-323_HandSoldering"
 			(at 120.65 121.92 0)
 			(effects
@@
 			)
 		)
-		(property "Footprint" "Diode:D_0603_1608Metric_Pad1.05x0.95mm_HandSolder"
+		(property "Footprint" "Diode_SMD:D_SOD-323_HandSoldering"
 			(at 124.46 49.53 0)
 			(effects
@@
 			)
 		)
-		(property "Footprint" "Diode:D_0603_1608Metric_Pad1.05x0.95mm_HandSolder"
+		(property "Footprint" "Diode_SMD:D_SOD-323_HandSoldering"
 			(at 104.14 73.66 0)
 			(effects
@@
 			)
 		)
-		(property "Footprint" "Diode:D_0603_1608Metric_Pad1.05x0.95mm_HandSolder"
+		(property "Footprint" "Diode_SMD:D_SOD-323_HandSoldering"
 			(at 124.46 121.92 0)
 			(effects
@@
 			)
 		)
-		(property "Footprint" "Diode:D_0603_1608Metric_Pad1.05x0.95mm_HandSolder"
+		(property "Footprint" "Diode_SMD:D_SOD-323_HandSoldering"
 			(at 166.37 97.79 0)
 			(effects
@@
 			)
 		)
-		(property "Footprint" "Diode:D_0603_1608Metric_Pad1.05x0.95mm_HandSolder"
+		(property "Footprint" "Diode_SMD:D_SOD-323_HandSoldering"
 			(at 181.61 97.79 0)
 			(effects
@@
 			)
 		)
-		(property "Footprint" "Diode:D_0603_1608Metric_Pad1.05x0.95mm_HandSolder"
+		(property "Footprint" "Diode_SMD:D_SOD-323_HandSoldering"
 			(at 142.24 121.92 0)
 			(effects
@@
 			)
 		)
-		(property "Footprint" "Diode:D_0603_1608Metric_Pad1.05x0.95mm_HandSolder"
+		(property "Footprint" "Diode_SMD:D_SOD-323_HandSoldering"
 			(at 166.37 121.92 0)
 			(effects
@@
 			)
 		)
-		(property "Footprint" "Diode:D_0603_1608Metric_Pad1.05x0.95mm_HandSolder"
+		(property "Footprint" "Diode_SMD:D_SOD-323_HandSoldering"
 			(at 146.05 97.79 0)
 			(effects
@@
 			)
 		)
-		(property "Footprint" "Diode:D_0603_1608Metric_Pad1.05x0.95mm_HandSolder"
+		(property "Footprint" "Diode_SMD:D_SOD-323_HandSoldering"
 			(at 205.74 73.66 0)
 			(effects
@@
 			)
 		)
-		(property "Footprint" "Diode:D_0603_1608Metric_Pad1.05x0.95mm_HandSolder"
+		(property "Footprint" "Diode_SMD:D_SOD-323_HandSoldering"
 			(at 120.65 49.53 0)
 			(effects
@@
 			)
 		)
-		(property "Footprint" "Diode:D_0603_1608Metric_Pad1.05x0.95mm_HandSolder"
+		(property "Footprint" "Diode_SMD:D_SOD-323_HandSoldering"
 			(at 104.14 97.79 0)
 			(effects
@@
 			)
 		)
-		(property "Footprint" "Diode:D_0603_1608Metric_Pad1.05x0.95mm_HandSolder"
+		(property "Footprint" "Diode_SMD:D_SOD-323_HandSoldering"
 			(at 185.42 121.92 0)
 			(effects
@@
 			)
 		)
-		(property "Footprint" "Diode:D_0603_1608Metric_Pad1.05x0.95mm_HandSolder"
+		(property "Footprint" "Diode_SMD:D_SOD-323_HandSoldering"
 			(at 100.33 146.05 0)
 			(effects
@@
 			)
 		)
-		(property "Footprint" "Diode:D_0603_1608Metric_Pad1.05x0.95mm_HandSolder"
+		(property "Footprint" "Diode_SMD:D_SOD-323_HandSoldering"
 			(at 100.33 73.66 0)
 			(effects
@@
 			)
 		)
-		(property "Footprint" "Diode:D_0603_1608Metric_Pad1.05x0.95mm_HandSolder"
+		(property "Footprint" "Diode_SMD:D_SOD-323_HandSoldering"
 			(at 104.14 49.53 0)
 			(effects

Commit message: Add TODOs for fixes for next version
Other:
- moved on the sheet: COL1, COL2, COL3, COL4, COL5, COL6, D1, D10, D11, D12, D13, D14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
